File: kicad/muikku42/_autosave-muikku42.kicad_sch (KiCad schematic)
At the start: 24 parts, among them U1 Raspberry_Pi_Pico, U2 TRRS, U3 TRRS

Commit message: New PCB design and new info
Everything has been updated, much simpler and cheaper design
Parts:
- S1, S10, S11, S12, S13, S14, S15, S16, S17, S18, S19, S2, S20, S21, S3, S4, S5, S6, S7, S8, S9: footprint kbd:CherryMX_MidHeight_Hotswap -> ScottoKeebs_Cutout:Cutout_MX_1.00u
Changed lines of the file:
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@@
 			)
 		)
-		(property "Footprint" "kbd:CherryMX_MidHeight_Hotswap"
+		(property "Footprint" "ScottoKeebs_Cutout:Cutout_MX_1.00u"
 			(at 36.83 81.28 0)
 			(effects
@@
 			)
 		)
-		(property "Footprint" "kbd:CherryMX_MidHeight_Hotswap"
+		(property "Footprint" "ScottoKeebs_Cutout:Cutout_MX_1.00u"
 			(at 86.36 45.72 0)
 			(effects
@@
 			)
 		)
-		(property "Footprint" "kbd:CherryMX_MidHeight_Hotswap"
+		(property "Footprint" "ScottoKeebs_Cutout:Cutout_MX_1.00u"
 			(at 55.88 63.5 0)
 			(effects
@@
 			)
 		)
-		(property "Footprint" "kbd:CherryMX_MidHeight_Hotswap"
+		(property "Footprint" "ScottoKeebs_Cutout:Cutout_MX_1.00u"
 			(at 76.2 45.72 0)
 			(effects
@@
 			)
 		)
-		(property "Footprint" "kbd:CherryMX_MidHeight_Hotswap"
+		(property "Footprint" "ScottoKeebs_Cutout:Cutout_MX_1.00u"
 			(at 76.2 63.5 0)
 			(effects
@@
 			)
 		)
-		(property "Footprint" "kbd:CherryMX_MidHeight_Hotswap"
+		(property "Footprint" "ScottoKeebs_Cutout:Cutout_MX_1.00u"
 			(at 46.99 81.28 0)
 			(effects
@@
 			)
 		)
-		(property "Footprint" "kbd:CherryMX_MidHeight_Hotswap"
+		(property "Footprint" "ScottoKeebs_Cutout:Cutout_MX_1.00u"
 			(at 45.72 45.72 0)
 			(effects
@@
 			)
 		)
-		(property "Footprint" "kbd:CherryMX_MidHeight_Hotswap"
+		(property "Footprint" "ScottoKeebs_Cutout:Cutout_MX_1.00u"
 			(at 55.88 45.72 0)
 			(effects
@@
 			)
 		)
-		(property "Footprint" "kbd:CherryMX_MidHeight_Hotswap"
+		(property "Footprint" "ScottoKeebs_Cutout:Cutout_MX_1.00u"
 			(at 66.04 26.67 0)
 			(effects
@@
 			)
 		)
-		(property "Footprint" "kbd:CherryMX_MidHeight_Hotswap"
+		(property "Footprint" "ScottoKeebs_Cutout:Cutout_MX_1.00u"
 			(at 66.04 45.72 0)
 			(effects
@@
 			)
 		)
-		(property "Footprint" "kbd:CherryMX_MidHeight_Hotswap"
+		(property "Footprint" "ScottoKeebs_Cutout:Cutout_MX_1.00u"
 			(at 86.36 26.67 0)
 			(effects
@@
 			)
 		)
-		(property "Footprint" "kbd:CherryMX_MidHeight_Hotswap"
+		(property "Footprint" "ScottoKeebs_Cutout:Cutout_MX_1.00u"
 			(at 55.88 26.67 0)
 			(effects
@@
 			)
 		)
-		(property "Footprint" "kbd:CherryMX_MidHeight_Hotswap"
+		(property "Footprint" "ScottoKeebs_Cutout:Cutout_MX_1.00u"
 			(at 66.04 63.5 0)
 			(effects
@@
 			)
 		)
-		(property "Footprint" "kbd:CherryMX_MidHeight_Hotswap"
+		(property "Footprint" "ScottoKeebs_Cutout:Cutout_MX_1.00u"
 			(at 76.2 26.67 0)
 			(effects
@@
 			)
 		)
-		(property "Footprint" "kbd:CherryMX_MidHeight_Hotswap"
+		(property "Footprint" "ScottoKeebs_Cutout:Cutout_MX_1.00u"
 			(at 35.56 63.5 0)
 			(effects
@@
 			)
 		)
-		(property "Footprint" "kbd:CherryMX_MidHeight_Hotswap"
+		(property "Footprint" "ScottoKeebs_Cutout:Cutout_MX_1.00u"
 			(at 35.56 26.67 0)
 			(effects
@@
 			)
 		)
-		(property "Footprint" "kbd:CherryMX_MidHeight_Hotswap"
+		(property "Footprint" "ScottoKeebs_Cutout:Cutout_MX_1.00u"
 			(at 35.56 45.72 0)
 			(effects
@@
 			)
 		)
-		(property "Footprint" "kbd:CherryMX_MidHeight_Hotswap"
+		(property "Footprint" "ScottoKeebs_Cutout:Cutout_MX_1.00u"
 			(at 57.15 81.28 0)
 			(effects
@@
 			)
 		)
-		(property "Footprint" "kbd:CherryMX_MidHeight_Hotswap"
+		(property "Footprint" "ScottoKeebs_Cutout:Cutout_MX_1.00u"
 			(at 45.72 63.5 0)
 			(effects
@@
 			)
 		)
-		(property "Footprint" "kbd:CherryMX_MidHeight_Hotswap"
+		(property "Footprint" "ScottoKeebs_Cutout:Cutout_MX_1.00u"
 			(at 86.36 63.5 0)
 			(effects
@@
 			)
 		)
-		(property "Footprint" "kbd:CherryMX_MidHeight_Hotswap"
+		(property "Footprint" "ScottoKeebs_Cutout:Cutout_MX_1.00u"
 			(at 45.72 26.67 0)
 			(effects
